Commit message: removed not working files, now skid steer mission works, lidar added to 4 wheel robot

File: urdf/mogi_bot.urdf (robot description, URDF)
Before this commit: robot mogi_bot, 9 links, 8 joints
Joints:
- joint base_footprint_joint: origin xyz=0.5 0 0.1 rpy=0 0 0 -> xyz=0.0 0.0 0.1 rpy=0 0 0

File: urdf/mogi_bot_skid_steer.urdf (robot description, URDF)
Before this commit: robot mogi_bot, 8 links, 7 joints
Links:
- added link scan_link, mass 1e-5; collision box size=0.1 0.1 0.1; visual mesh filename=package://erl_assignment_2/meshes/lidar.dae
Joints:
- added joint scan_joint: type fixed, parent base_link, child scan_link, origin xyz=0 0 0.12 rpy=0 0 0, axis 0 1 0
